Commit message: updated static tf

File: mini_alpha_description/urdf/base.urdf (robot description, URDF)
Before this commit: robot mini_alpha, 11 links, 10 joints
Joints:
- joint heave_port_thruster_joint: origin xyz=-0.381 0.11 0.0 rpy=0.0 1.5717 0.0 -> xyz=-0.381 0.11 0.0 rpy=0.0 1.57079 0.0
- joint heave_starboard_thruster_joint: origin xyz=-0.381 -0.11 0.0 rpy=0.0 1.5717 0.0 -> xyz=-0.381 -0.11 0.0 rpy=0.0 1.57079 0.0
- joint imu_joint: origin xyz=0.0 -0.0 0.0 rpy=0.0 0.0 0.0 -> xyz=0.0 -0.0 0.0 rpy=0.0 0.0 3.1415926

Commit message: commit after allen harbor

File: mini_alpha_description/urdf/base.urdf (robot description, URDF)
Before this commit: robot mini_alpha, 11 links, 10 joints
Joints:
- joint base_link: origin xyz=-0.0 0.0 0.0 rpy=0.0 0.0 0.0 -> xyz=-0.3 0.0 0.0 rpy=0.0 0.0 0.0
- joint heave_port_thruster_joint: origin xyz=-0.381 0.11 0.0 rpy=0.0 1.57079 0.0 -> xyz=-0.2 0.11 0.0 rpy=0.0 1.57079 0.0
- joint heave_starboard_thruster_joint: origin xyz=-0.381 -0.11 0.0 rpy=0.0 1.57079 0.0 -> xyz=-0.2 -0.11 0.0 rpy=0.0 1.57079 0.0
- joint imu_joint: origin xyz=0.0 -0.0 0.0 rpy=0.0 0.0 3.1415926 -> xyz=-0.1 0.0 0.0 rpy=0.0 0.0 3.1415926
- joint surge_port_thruster_joint: origin xyz=-0.53 0.11 0.0 rpy=0.0 0.0 0.0 -> xyz=-0.3 0.11 0.0 rpy=0.0 0.0 0.0
- joint surge_starboard_thruster_joint: origin xyz=-0.53 -0.11 0.0 rpy=0.0 0.0 0.0 -> xyz=-0.3 -0.11 0.0 rpy=0.0 0.0 0.0
